File: Kicad/keyboard/TutorialKeyboard/tutorial_keyboard/tutorial_keyboard.sch (KiCad schematic (older format))
At the start: 113 parts, among them J1 USB_C_Receptacle_USB2.0, K1 KEYSW, K10 KEYSW, K11 KEYSW, K12 KEYSW, K13 KEYSW, K14 KEYSW, K15 KEYSW, K16 KEYSW, K17 KEYSW, K18 KEYSW, K19 KEYSW, K2 KEYSW, K20 KEYSW, K21 KEYSW, K22 KEYSW, K23 KEYSW, K24 KEYSW, K25 KEYSW, K26 KEYSW, K27 KEYSW, K28 KEYSW, K29 KEYSW, K3 KEYSW, K30 KEYSW, K31 KEYSW, K32 KEYSW, K33 KEYSW, K34 KEYSW, K35 KEYSW, K36 KEYSW, K37 KEYSW, K38 KEYSW, K39 KEYSW, K4 KEYSW, K40 KEYSW, K41 KEYSW, K42 KEYSW, K43 KEYSW, K44 KEYSW, K45 KEYSW, K46 KEYSW, K47 KEYSW, K5 KEYSW, K6 KEYSW, K7 KEYSW, K8 KEYSW, K9 KEYSW, SW1 SW_PUSH, U1 ATMEGA32U4, X1 XTAL

Commit message: up to routing section
Parts:
- J1: footprint keebs:Mx_Alps_100 -> Type-C:USB_C_GCT_USB4085
Changed lines of the file:
@@
 EESchema Schematic File Version 4
+LIBS:tutorial_keyboard-cache
 EELAYER 29 0
 EELAYER END
@@
 F 0 "J1" H 3357 3317 50  0000 C CNN
 F 1 "USB_C_Receptacle_USB2.0" H 3357 3226 50  0000 C CNN
-F 2 "keebs:Mx_Alps_100" H 3400 2450 50  0001 C CNN
+F 2 "Type-C:USB_C_GCT_USB4085" H 3400 2450 50  0001 C CNN
 F 3 "https://www.usb.org/sites/default/files/documents/usb_type-c.zip" H 3400 2450 50  0001 C CNN
 	1    3250 2450
